File: hardware_design/Peaks.sch (KiCad schematic (older format))
At the start: 69 parts, among them J1 in1, J2 in2, J3 Eurorack Power, J4 out1, J5 out2, J8 Conn_01x07, Q1 2N3904, Q2 2N3904, SW1 SW_Dual, SW2 SW_Mode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

Commit message: Remixed hardware.
Skiff friendly (50cm depth) PCB.
Revert to using more standard KiCad footprints.
Use a 5.1V Zener diode for PWM scaling.
Parts:
- added J10, J9: Conn_01x03, Connector_PinHeader_2.54mm:PinHeader_1x03_P2.54mm_Vertical, symbol Connector_Generic:Conn_01x03
- added J11, J12, J13, J14, J15: Conn_01x02, Connector_PinHeader_2.54mm:PinHeader_1x02_P2.54mm_Vertical, symbol Connector_Generic:Conn_01x02
- D10: value 3.6 -> 5.1; footprint Personal:D_DO-35_SOD27_P2.54mm_Vertical_AnodeUp_Large_Pads -> Resistor_THT:R_Axial_DIN0204_L3.6mm_D1.6mm_P7.62mm_Horizontal
- R1, R12, R13, R19, R20, R3, R7: footprint Personal:R_Axial_DIN0204_L3.6mm_D1.6mm_P2.54mm_Vertical_Large_Pads -> Resistor_THT:R_Axial_DIN0207_L6.3mm_D2.5mm_P7.62mm_Horizontal
- R10, R11, R2, R4, R5, R8: footprint Personal:R_Axial_DIN0204_L3.6mm_D1.6mm_P2.54mm_Vertical_Large_Pads -> Resistor_THT:R_Axial_DIN0204_L3.6mm_D1.6mm_P7.62mm_Horizontal
- R14: value 15k -> 21k; footprint Personal:R_Axial_DIN0204_L3.6mm_D1.6mm_P2.54mm_Vertical_Large_Pads -> Resistor_THT:R_Axial_DIN0204_L3.6mm_D1.6mm_P7.62mm_Horizontal
- R15, R17, R22, R23: footprint Personal:R_Axial_DIN0204_L3.6mm_D1.6mm_P7.62mm_Horizontal_Large_Pads -> Resistor_THT:R_Axial_DIN0207_L6.3mm_D2.5mm_P7.62mm_Horizontal
- R16: value 15k -> 21k; footprint Personal:R_Axial_DIN0204_L3.6mm_D1.6mm_P7.62mm_Horizontal_Large_Pads -> Resistor_THT:R_Axial_DIN0207_L6.3mm_D2.5mm_P7.62mm_Horizontal
- R18, R21, R24, R25, R26, R27, R28, R6, R9: footprint Personal:R_Axial_DIN0204_L3.6mm_D1.6mm_P2.54mm_Vertical_Large_Pads -> Resistor_THT:R_Axial_DIN0204_L3.6mm_D1.6mm_P2.54mm_Vertical
- RV1, RV2, RV3, RV4: footprint Personal:Potenciometro -> Potentiometer_THT:Potentiometer_Alps_RK097_Single_Horizontal
- U3: value 78l05 -> 78L05
Connections:
- net labels added: 3.3V, REF_-5V
- net labels removed: +3.3V, REF_-3.6
- wire segments 148 -> 178
- no-connect marks 0 -> 2
Other:
- note added: "*If you want to recalculate these resistors \nbecause of a different zener value use this ecuation:\n0.1 = 33(-Vzener/R + 1.65/6.8)\n\nFor 5.1V Zener, R14 = 21k\nFor 3.3V Zener, R14 = 14k\nFon 3.6V Zener, R14 = 15k"
- note removed: "*If you want to recalculate these resistors \nbecause of a different zener value use this ecuation:\n0.1 = 33(-Vzener/R + 1.65/6.8)"
- moved on the sheet: C10, D1, D2, D3, D4, D5, D6, D7, J1, J2, J8, Q1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
